File: PCB/Flasher/Flasher.kicad_sch (KiCad schematic)
At the start: 48 parts, among them J1 1x5, J2 TC2030-USB-NL, J3 Reset, Q1 BSS138PS, U1 TPS562246, U4 ESP32-S3-MINI-1

Commit message: Start PCb
Parts:
- removed D2, D3: ~, RevK:DFN1006-2L, symbol RevK:ES05D1MC10
- removed D4: D, RevK:D_0402, symbol Device:D
- removed J1: 1x5, RevK:JST_EH_S5B-EH_1x05_P2.50mm_Horizontal, symbol Connector_Generic:Conn_01x05
- removed J2: TC2030-USB-NL, RevK:Tag-Connect_TC2030-IDC-NL_2x03_P1.27mm_Vertical, symbol RevK:TC2030-USB-NL-LB
- removed Q1: BSS138PS, RevK:SOT-363_SC-70-6, symbol RevK:BSS138PS
- removed R1, R2: 10k, RevK:R_0201, symbol Device:R
- removed TP1: TestPoint, RevK:1x2-Hole, symbol Connector:TestPoint
- removed V1, V2: ~, RevK:VCUT70N, symbol RevK:VCUT
Other:
- note removed: "2/6 are loop back test via TC2030m cable."
- note removed: "A cap Tx to GND seems obvious But experiments show it makes it way more noisy!"
- note removed: "Careful routing of Rx line to avoid the regulator"
- title: Daikin ESP32-PICO-MINI module -> Flasher
- moved on the sheet: D1

Commit message: Parts
Parts:
- removed TP10, TP2, TP3, TP4, TP5, TP6, TP7, TP8, TP9: TestPoint, RevK:PAD-2mm, symbol Connector:TestPoint
- added C13: 100nF, RevK:C_0402, symbol Device:C
- added C14, C15, C16: 100nF, RevK:C_0201, symbol Device:C
- added D10, D2, D3, D4, D5, D6, D7, D8, D9: XL-1010RGBC-WS2812B, RevK:SMD1010, symbol RevK:WS2812B-1mm
- added J2, J3: Wago, RevK:WAGO-2060-453-998-404, symbol Connector_Generic:Conn_01x03
- added J4: USB-C-Socket-V, RevK:USB-C-Socket-H, symbol RevK:USB-C-Socket-H
- added J5: TF_PUSH, RevK:TF_PUSH, symbol RevK:TF_PUSH
- added R10, R9: 27R, RevK:R_0201, symbol Device:R
- added R11, R12, R13, R14, R15, R5, R6: 10K, RevK:R_0201, symbol Device:R
- added R7, R8: 5K1, RevK:R_0201, symbol Device:R
- added U3: FT231XQ, RevK:QFN-20-1EP_4x4mm_P0.5mm_EP2.5x2.5mm, symbol RevK:FT231XQ
- added U4: TPS22916CNYFPR, RevK:WCSP-4-0.78x0.78, symbol RevK:TPS22916
- renumbered C17 to C1, C4 to C10, C5 to C11, C7 to C12, C3 to C2, C16 to C3, C6 to C4, C18 to C5, C19 to C6, C15 to C7, C1 to C8, C2 to C9, FID2 to FID1, FID3 to FID2, J3 to J1, R5 to R1, R3 to R2, R6 to R3, R8 to R4, U4 to U1, U1 to U2, V5 to V1, V3 to V2, V4 to V3, V6 to V4
Connections:
- net +3.3V: now also C14.1, C15.1, C16.1, D10.2 (+), D2.2 (+), D3.2 (+), D4.2 (+), D5.2 (+), D6.2 (+), D7.2 (+), D8.2 (+), D9.2 (+), J5.4 (VDD), R11.1, R12.1, R13.1, R14.1, R15.1, R5.1, R6.1
- net D+: now also J2.1 (Pin_1)
- net D-: now also J3.3 (Pin_3)
- net GND: now also C13.2, C14.2, C15.2, C16.2, D10.3 (-), D2.3 (-), D3.3 (-), D4.3 (-), D5.3 (-), D6.3 (-), D7.3 (-), D8.3 (-), D9.3 (-), J2.2 (Pin_2), J4.A1 (GND), J4.A12 (GND), J4.B1 (GND), J4.B12 (GND), J4.S1 (SHIELD), J5.6 (VSS), J5.S (SHIELD), R7.2, R8.1, U3.13 (GND), U3.2 (~{RI}), U3.21 (GND), U3.3 (GND), U3.4 (~{DSR}), U3.5 (~{DCD}), U3.6 (~{CTS}), U4.B1 (GND); no longer U1.16 (GPIO12), U1.17 (GPIO13), U1.18 (GPIO14), U1.19 (GPIO15), U1.20 (GPIO16), U1.21 (GPIO17), U1.22 (GPIO18), U1.28 (GPIO33)
- net RST: now also U3.19 (~{RTS})
- net at D1.1 (O): now also D2.4 (I)
- net PWR: now reaches U1.15 (GPIO11)
- net PWR: now also U4.B2 (ON)
- net TXD: now reaches U1.39 (GPIO43)
- net TXD: now also U3.1 (RXD)
- net GPIO0: now reaches U1.4 (GPIO0)
- net GPIO0: now also U3.18 (~{DTR})
- net RXD: now reaches U1.40 (GPIO44)
- net RXD: now also U3.17 (TXD)
- net RX: no longer names the net of U1.29 (GPIO34)
- net TX: no longer names the net of U1.30 (GPIO48)
- new net: J4.A5 (CC1), R7.1
- new net: J4.B5 (CC2), R8.2
- new net: J4.A6 (D+), J4.B6 (D+), R10.1
- new net: R10.2, U3.8 (USBDP)
- new net: D5.1 (O), D6.4 (I)
- new net: D4.1 (O), D5.4 (I)
- new net: J4.A7 (D-), J4.B7 (D-), R9.1
- new net: R9.2, U3.9 (USBDM)
- new net: D6.1 (O), D7.4 (I)
- new net: C13.1, U3.10 (3V3OUT), U3.11 (~{RESET}), U3.20 (VCCIO)
- new net: J2.3 (Pin_3), J3.2 (Pin_2)
- new net: D10.4 (I), D9.1 (O)
- new net: D2.1 (O), D3.4 (I)
- new net: J3.1 (Pin_1), U4.A1 (VOUT)
- new net: D7.1 (O), D8.4 (I)
- new net: D3.1 (O), D4.4 (I)
- new net: D8.1 (O), D9.4 (I)
- new net SDCD: J5.9 (CD), R5.2, U1.22 (GPIO18)
- new net SDCLK: J5.5 (CLK), R12.2, U1.19 (GPIO15)
- new net SDCMD: J5.3 (CMD), R13.2, U1.18 (GPIO14)
- new net SDDAT0: J5.7 (DAT0), R11.2, U1.20 (GPIO16)
- new net SDDAT1: J5.8 (DAT1), R6.2, U1.21 (GPIO17)
- new net SDDAT2: J5.1 (DAT2), R15.2, U1.16 (GPIO12)
- new net SDDAT3: J5.2 (DAT3/CD), R14.2, U1.17 (GPIO13)
- new net VBUS: J4.A4 (VBUS), J4.A9 (VBUS), J4.B4 (VBUS), J4.B9 (VBUS), U3.12 (VCC), U4.A2 (VIN)
- no-connect marks 25 -> 28
Other:
- note added: "Configure FTDI - Inverted RTS"
- note added: "TC2030"
- note removed: "Regulator block - IC rated 3.3V 2A, but thermal considerations are based on typical usage."
- moved on the sheet: C4, D1, FID1, FID2, J1, R2, U1
