File: PCB/Flasher2/Flasher.kicad_pcb (KiCad board)
At the start: 2 copper layers, 70 x 70 mm, 63 parts, among them J1 Reset, J2 RJ12, J3 USB, J4 USB-C-Socket-V, J5 TF_PUSH, J6 LCD, SW3 SW_Push_SPDT, U1 ESP32-S3-MINI-1, U2 TPS562246, U3 FT231XQ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

Commit message: Minor tweaks
Parts:
- moved J2 0.50 mm to (127.5, 44.0)
Routing:
- net Net-(D10-O): track 65.9 -> 63.7 mm
- net LOOP: track 39.4 -> 40.0 mm
- net D+: track 43.7 -> 44.2 mm
